File: hardware/Main_Project.kicad_sch (KiCad schematic)
At the start: 48 parts, among them J1 A_Motor, J2 B_Motor, SW1 Power_Switch, U1 L7805, U2 L298N, U3 L298N

Commit message: Added example text
Other:
- note added: "Example Text"

Commit message: Added footprints for Colour sensor and reorganized libraries
Parts:
- D2: value D -> 1N4004
- D3: value LED -> LED_Red
- D4: value LED -> LED_Yellow
- R1, R2: value 2.2k -> 470R
Changed lines of the file:
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@@
       (effects (font (size 1.27 1.27)) (justify left))
     )
-    (property "Value" "2.2k" (at 64.008 86.3021 0)
+    (property "Value" "470R" (at 64.008 86.3021 0)
       (effects (font (size 1.27 1.27)) (justify left))
     )
@@
       (effects (font (size 1.27 1.27)))
     )
-    (property "Value" "D" (at 80.01 33.8399 0)
+    (property "Value" "1N4004" (at 80.01 33.8399 0)
       (effects (font (size 1.27 1.27)))
     )
@@
       (effects (font (size 1.27 1.27)) (justify left))
     )
-    (property "Value" "2.2k" (at 90.678 43.1221 0)
+    (property "Value" "470R" (at 90.678 43.1221 0)
       (effects (font (size 1.27 1.27)) (justify left))
     )
@@
       (effects (font (size 1.27 1.27)) (justify right))
     )
-    (property "Value" "LED" (at 65.151 95.5096 90)
+    (property "Value" "LED_Yellow" (at 65.151 95.5096 90)
       (effects (font (size 1.27 1.27)) (justify right))
     )
@@
       (effects (font (size 1.27 1.27)) (justify right))
     )
-    (property "Value" "LED" (at 91.821 52.3296 90)
+    (property "Value" "LED_Red" (at 91.821 52.3296 90)
       (effects (font (size 1.27 1.27)) (justify right))
     )

Commit message: Changed PCB slightly
Parts:
- added U4: ~, TDP3KICAD:Adafruit_Flora_Sensor, symbol TDP3KICAD:Adafruit_Flora_Sensor
Changed lines of the file:
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@@
+    )
+  )
+  (symbol (lib_id "TDP3KICAD:Adafruit_Flora_Sensor") (at 212.09 130.81 0) (unit 1)
+    (in_bom yes) (on_board yes) (dnp no) (fields_autoplaced)
+    (property "Reference" "U4" (at 216.535 130.81 0)
+      (effects (font (size 1.27 1.27)) (justify left))
+    )
+    (property "Value" "~" (at 212.09 130.81 0)
+      (effects (font (size 1.27 1.27)))
+    )
+    (property "Footprint" "TDP3KICAD:Adafruit_Flora_Sensor" (at 212.09 130.81 0)
+      (effects (font (size 1.27 1.27)) hide)
+    )
+    (property "Datasheet" "" (at 212.09 130.81 0)
+      (effects (font (size 1.27 1.27)) hide)
+    )
+    (pin "1")
+    (pin "2")
+    (pin "3")
+    (pin "4")
+    (pin "5")
+    (pin "6")
+    (instances
+      (project "Main_Project"
+        (path "/49595465-104c-4a4c-848b-e24eebb1e8d2"
+          (reference "U4") (unit 1)
+        )
+      )
     )
   )
