File: hardware/_autosave-Main_Project.kicad_sch (KiCad schematic)
At the start: 53 parts, among them J1 A_Motor, J2 B_Motor, J3 Power_Outputs, U1 L7805, U2 L298N, U4 L298N

Commit message: Created Power PCB
Parts:
- U1: footprint Package_TO_SOT_THT:TO-220-3_Vertical -> Package_TO_SOT_THT:TO-220-3_Horizontal_TabDown
Changed lines of the file:
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@@
       (effects (font (size 1.27 1.27)))
     )
-    (property "Footprint" "Package_TO_SOT_THT:TO-220-3_Vertical" (at 38.735 82.55 0)
+    (property "Footprint" "Package_TO_SOT_THT:TO-220-3_Horizontal_TabDown" (at 38.735 82.55 0)
       (effects (font (size 1.27 1.27) italic) (justify left) hide)
     )
