File: hardware/Main_Project.kicad_pcb (KiCad board)
At the start: 2 copper layers, 41.1 x 40.8 mm, 53 parts, among them J1 A_Motor, J2 B_Motor, J3 Power_Outputs, U1 L7805, U2 L298N, U4 L298N

Commit message: Motor Board
Parts:
- removed C6, C8, C9: 4.7uF, Capacitor_THT:CP_Radial_D10.0mm_P5.00mm
- removed C7: 100nF, Capacitor_THT:C_Disc_D8.0mm_W2.5mm_P5.00mm
- removed D13, D14, D15, D16, D17, D18, D19, D20: D, Diode_THT:D_A-405_P10.16mm_Horizontal
- removed R10, R5, R6, R9: 1k, Resistor_THT:R_Axial_DIN0207_L6.3mm_D2.5mm_P10.16mm_Horizontal
- removed R3, R4, R7, R8: 10k, Resistor_THT:R_Axial_DIN0207_L6.3mm_D2.5mm_P10.16mm_Horizontal
- removed U4: L298N, Package_TO_SOT_THT:TO-220-15_P2.54x2.54mm_StaggerOdd_Lead4.58mm_Vertical
- added H10: HeatsinkMounting, new_winterbloom:M3_Heatsink_Mounting, F.Cu at (252.2, 67.6)
- added H5: MountingHole, MountingHole:MountingHole_3mm, F.Cu at (216.2, 44.2)
- added H6: MountingHole, MountingHole:MountingHole_3mm, F.Cu at (263.4, 44.2)
- added H7: MountingHole, MountingHole:MountingHole_3mm, F.Cu at (263.4, 87.1)
- added H8: MountingHole, MountingHole:MountingHole_3mm, F.Cu at (216.2, 87.1)
- added H9: HeatsinkMounting, new_winterbloom:M3_Heatsink_Mounting, F.Cu at (226.8, 67.6)
- added J4: Motor_Control, Connector_Molex:Molex_KK-396_5273-06A_1x06_P3.96mm_Vertical, F.Cu at (257.8, 46.5)
- added J5: Motor_Power, TerminalBlock:TerminalBlock_bornier-3_P5.08mm, F.Cu at (232.7, 44.7)
- C5: footprint Capacitor_THT:CP_Radial_D10.0mm_P5.00mm -> Capacitor_THT:CP_Radial_D8.0mm_P3.50mm
- J1: value A_Motor -> Motors_R
- J2: value B_Motor -> Motors_L
- moved J1 158.2 mm to (258.8, 94.5)
- moved D11 154.8 mm to (254.0, 96.3), turned to 90 degrees
- moved D7 152.5 mm to (250.4, 86.1), turned to -90 degrees
- moved D12 147.2 mm to (246.9, 96.3), turned to 90 degrees
- moved D8 144.7 mm to (243.3, 86.1), turned to -90 degrees
- moved D9 138.9 mm to (236.2, 96.3), turned to 90 degrees
- moved D5 137.2 mm to (232.7, 86.1), turned to -90 degrees
- moved D10 131.1 mm to (229.1, 96.3), turned to 90 degrees
- moved D6 129.2 mm to (225.6, 86.1), turned to -90 degrees
- moved C4 127.2 mm to (239.8, 86.7), turned to -90 degrees
- moved C5 121.7 mm to (237.9, 59.7)
- moved J2 117.9 mm to (215.6, 94.5)
- moved U2 107.5 mm to (230.6, 77.5)
- moved C3 70.7 mm to (170.4, 60.9), turned to -90 degrees
- moved U3 41.3 mm to (91.9, 79.2)
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Connections:
- J1 pad 1: Net-(D5-A) -> Net-(D11-K)
- J1 pad 2: Net-(D10-K) -> Net-(D12-K)
- J2 pad 1: Net-(D13-A) -> Net-(D5-A)
- J2 pad 2: Net-(D14-A) -> Net-(D10-K)
- U2 pad 1: Net-(U2-SENSE_A) -> GND
- U2 pad 10: A_Motor3 -> /R_1
- U2 pad 11: Net-(U2-EnB) -> /R_Enable
- U2 pad 12: A_Motor4 -> /R_2
- U2 pad 15: Net-(U2-SENSE_B) -> GND
- U2 pad 5: A_Motor1 -> /L_1
- U2 pad 6: Net-(U2-EnA) -> /L_Enable
- U2 pad 7: A_Motor2 -> /L_2
Routing:
- net +12V: track 38.4 -> 185.8 mm
- net +5V: track 41.1 -> 124.1 mm, vias 0 -> 1
- net /L_2: track 0.00 -> 73.1 mm, vias 0 -> 1
- net /L_1: track 0.00 -> 69.8 mm, vias 0 -> 1
- net /R_Enable: track 0.00 -> 65.6 mm, vias 0 -> 1
- net Net-(D5-A): track 0.00 -> 52.4 mm
- net Net-(D12-K): track 0.00 -> 50.7 mm
- net Net-(D10-K): track 0.00 -> 32.3 mm
- net Net-(D11-K): track 0.00 -> 31.6 mm
- net /L_Enable: track 0.00 -> 30.4 mm
- net /R_1: track 0.00 -> 27.8 mm
- net /R_2: track 0.00 -> 26.4 mm
Other:
- board size 41.1 x 40.8 mm -> 109.8 x 58.2 mm
- board text added: "Heatsink hole size = 3mm"
- board text added: "L1"

Commit message: Colour Sensor board added and adjusted
Parts:
- added C6: 4.7uF, Capacitor_THT:CP_Radial_D8.0mm_P3.50mm, F.Cu at (120.3, 83.6)
- added H11: MountingHole, MountingHole:MountingHole_3mm, F.Cu at (56.1, 114.6)
- added H12: MountingHole, MountingHole:MountingHole_3mm, F.Cu at (119.9, 114.6)
- added H13: MountingHole, MountingHole:MountingHole_3mm, F.Cu at (56.1, 35.1)
- added H14: MountingHole, MountingHole:MountingHole_3mm, F.Cu at (119.9, 35.1)
- added H15: MountingHole, MountingHole:MountingHole_3mm, F.Cu at (29.2, 122.9)
- added H16: MountingHole, MountingHole:MountingHole_3mm, F.Cu at (29.0, 27.9)
- added H17: MountingHole, MountingHole:MountingHole_3mm, F.Cu at (144.5, 125.5)
- added H18: MountingHole, MountingHole:MountingHole_3mm, F.Cu at (174.5, 125.5)
- added H19: MountingHole, MountingHole:MountingHole_3mm, F.Cu at (144.5, 155.4)
- added H20: MountingHole, MountingHole:MountingHole_3mm, F.Cu at (174.5, 155.4)
- added H21: MountingHole, MountingHole:MountingHole_5.3mm_M5, F.Cu at (198.1, 133.3)
- added H22: MountingHole, MountingHole:MountingHole_5.3mm_M5, F.Cu at (198.1, 147.6)
- added J10: BBBBBBBONUSROUND, Connector_Molex:Molex_KK-254_AE-6410-04A_1x04_P2.54mm_Vertical, F.Cu at (55.9, 94.5)
- added J11: Power_Distro, TerminalBlock:TerminalBlock_bornier-4_P5.08mm, F.Cu at (29.1, 100.3)
- added J12: Power_Distro, TerminalBlock:TerminalBlock_bornier-4_P5.08mm, F.Cu at (29.0, 35.1)
- added J13: Power_Distro, TerminalBlock:TerminalBlock_bornier-4_P5.08mm, F.Cu at (29.1, 78.7)
- added J14: Power_Distro, TerminalBlock:TerminalBlock_bornier-4_P5.08mm, F.Cu at (29.1, 57.1)
- added J15: Color_Sensor, Connector_Molex:Molex_KK-254_AE-6410-04A_1x04_P2.54mm_Vertical, F.Cu at (184.1, 129.8)
- added J16: Color_Sensor, Connector_Molex:Molex_KK-254_AE-6410-04A_1x04_P2.54mm_Vertical, F.Cu at (184.1, 143.5)
- added J6: Motor_Power, TerminalBlock:TerminalBlock_bornier-3_P5.08mm, F.Cu at (119.3, 65.3)
- added J7: Motor_Control, Connector_Molex:Molex_KK-254_AE-6410-06A_1x06_P2.54mm_Vertical, F.Cu at (56.1, 67.8)
- added J8: Color_Sensor, Connector_Molex:Molex_KK-254_AE-6410-04A_1x04_P2.54mm_Vertical, F.Cu at (118.9, 57.7)
- added J9: Magnet?, Connector_Molex:Molex_KK-254_AE-6410-04A_1x04_P2.54mm_Vertical, F.Cu at (56.1, 81.8)
- J4: footprint Connector_Molex:Molex_KK-396_5273-06A_1x06_P3.96mm_Vertical -> Connector_Molex:Molex_KK-254_AE-6410-06A_1x06_P2.54mm_Vertical
- moved U3 91.2 mm to (159.5, 140.4)
- moved FRDM1 6.84 mm to (87.4, 70.4)
- moved J4 3.09 mm to (255.8, 44.2)
- moved H2 0.84 mm to (194.8, 44.2)
- moved H1 0.40 mm to (160.5, 44.2)
- moved H4 0.14 mm to (194.6, 78.2)
- moved H3 0.12 mm to (160.5, 78.1)
- moved C3 0.08 mm to (170.4, 61.0)
Connections:
- FRDM1 pad A4: unconnected-(FRDM1-A4/PTC2-PadA4) -> /SDA
- FRDM1 pad A5: unconnected-(FRDM1-A5/PTC1-PadA5) -> /SCL
- FRDM1 pad D1: unconnected-(FRDM1-D1/PTA2-PadD1) -> /L_Enable
- FRDM1 pad D10: unconnected-(FRDM1-D10/PTD0-PadD10) -> Net-(FRDM1-D10/PTD0)
- FRDM1 pad D11: unconnected-(FRDM1-D11/PTD2-PadD11) -> Net-(FRDM1-D11/PTD2)
- FRDM1 pad D12: unconnected-(FRDM1-D12/PTD3-PadD12) -> Net-(FRDM1-D12/PTD3)
- FRDM1 pad D13: unconnected-(FRDM1-D13/PTD1-PadD13) -> Net-(FRDM1-D13/PTD1)
- FRDM1 pad D14: unconnected-(FRDM1-SDA/PTE0-PadD14) -> Net-(FRDM1-SDA/PTE0)
- FRDM1 pad D15: unconnected-(FRDM1-SCL/PTE1-PadD15) -> Net-(FRDM1-SCL/PTE1)
- FRDM1 pad D2: unconnected-(FRDM1-D2/PTD4-PadD2) -> /R_1
- FRDM1 pad D3: unconnected-(FRDM1-D3/PTA12-PadD3) -> /R_2
- FRDM1 pad D4: unconnected-(FRDM1-D4/PTA4-PadD4) -> /R_Enable
- FRDM1 pad D5: unconnected-(FRDM1-D5/PTA5-PadD5) -> /L_2
- FRDM1 pad D6: unconnected-(FRDM1-D6/PTC8-PadD6) -> /L_1
- FRDM1 pad D8: unconnected-(FRDM1-D8/PTA13-PadD8) -> Net-(FRDM1-D8/PTA13)
- FRDM1 pad D9: unconnected-(FRDM1-D9/PTD5-PadD9) -> Net-(FRDM1-D9/PTD5)
- FRDM1 pad GND0: unconnected-(FRDM1-PadGND0) -> GND
- FRDM1 pad GND1: unconnected-(FRDM1-PadGND1) -> GND
- FRDM1 pad P3V3: unconnected-(FRDM1-3V3-PadP3V3) -> +3V3
- FRDM1 pad VIN: unconnected-(FRDM1-PadVIN) -> Net-(J6-Pin_2)
- U3 pad 1: unconnected-(U3-3V3-Pad1) -> Net-(J15-Pin_1)
- U3 pad 2: unconnected-(U3-SDA_A-Pad2) -> Net-(J15-Pin_2)
- U3 pad 3: unconnected-(U3-SCL_A-Pad3) -> Net-(J15-Pin_3)
- U3 pad 4: unconnected-(U3-GND-Pad4) -> GND
- U3 pad 5: unconnected-(U3-SCL_B-Pad5) -> Net-(J15-Pin_3)
- U3 pad 6: unconnected-(U3-SDA_B-Pad6) -> Net-(J15-Pin_2)
Routing:
- net +3V3: track 0.00 -> 145.4 mm
- net +12V: track 185.8 -> 285.9 mm
- net +5V: track 124.1 -> 203.9 mm
- net Net-(J15-Pin_1): track 0.00 -> 70.8 mm
- net Net-(J15-Pin_2): track 0.00 -> 55.1 mm
- net Net-(J15-Pin_3): track 0.00 -> 54.9 mm
- net Net-(J6-Pin_2): track 0.00 -> 22.3 mm
- net GND: track 0.00 -> 15.2 mm
- net /R_2: track 26.4 -> 36.8 mm
- net /L_1: track 69.8 -> 80.1 mm
- net /R_Enable: track 65.6 -> 75.4 mm
- net /L_2: track 73.1 -> 82.8 mm
- net /R_1: track 27.8 -> 36.8 mm
- net Net-(FRDM1-SDA/PTE0): track 0.00 -> 8.40 mm
- net Net-(FRDM1-SCL/PTE1): track 0.00 -> 8.40 mm
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Other:
- board size 109.8 x 58.2 mm -> 246.8 x 135.9 mm
- board text added: "3V3"
- board text added: "Colour Sensor"
- board text added: "Colour Sensor Board"
- board text added: "Extra"
- board text added: "Motor Driver"
- board text removed: "Extra Footprints Please ignore"

Commit message: Updated Colour Sensor Board to fit properly
Routing:
- net Net-(J15-Pin_1): track 70.8 -> 45.9 mm
- net GND: track 15.2 -> 0.00 mm, vias 0 -> 1

Commit message: Magnet board
Parts:
- added C7: 4.7uF, Capacitor_THT:CP_Radial_D8.0mm_P3.50mm, F.Cu at (252.3, 135.9)
- added D13: 1N4004, Diode_THT:D_A-405_P10.16mm_Horizontal, F.Cu at (248.9, 152.1)
- added H23: HeatsinkMounting, new_winterbloom:M3_Heatsink_Mounting, F.Cu at (266.2, 142.7)
- added H24: HeatsinkMounting, new_winterbloom:M3_Heatsink_Mounting, F.Cu at (241.6, 142.7)
- added H25: MountingHole, MountingHole:MountingHole_3mm, F.Cu at (236.7, 126.2)
- added H26: MountingHole, MountingHole:MountingHole_3mm, F.Cu at (270.8, 126.2)
- added H27: MountingHole, MountingHole:MountingHole_3mm, F.Cu at (270.8, 160.3)
- added H28: MountingHole, MountingHole:MountingHole_3mm, F.Cu at (236.7, 160.3)
- added J17: Magnet, TerminalBlock:TerminalBlock_bornier-2_P5.08mm, F.Cu at (251.5, 159.5)
- added J18: FRDM input, Connector_Molex:Molex_KK-254_AE-6410-02A_1x02_P2.54mm_Vertical, F.Cu at (261.1, 127.0)
- added J19: Magnet_Power, TerminalBlock:TerminalBlock_bornier-3_P5.08mm, F.Cu at (253.7, 127.0)
- added Q2: BC547, Package_TO_SOT_THT:TO-92_Inline_Wide, F.Cu at (247.1, 160.7)
- added Q3: IRF540N, Package_TO_SOT_THT:TO-220-3_Vertical, F.Cu at (251.5, 147.0)
- added R3: 10k, Resistor_THT:R_Axial_DIN0207_L6.3mm_D2.5mm_P10.16mm_Horizontal, F.Cu at (235.0, 155.4)
- added R4: 1k, Resistor_THT:R_Axial_DIN0207_L6.3mm_D2.5mm_P10.16mm_Horizontal, F.Cu at (235.0, 152.1)
- added R5: Current_Limit, Resistor_THT:R_Axial_DIN0207_L6.3mm_D2.5mm_P10.16mm_Horizontal, F.Cu at (263.9, 162.1)
Routing:
- net Net-(J18-Pin_2): track 0.00 -> 55.7 mm
- net +5V: track 203.9 -> 240.0 mm
- net +12V: track 285.9 -> 321.4 mm
- net Net-(Q2-C): track 0.00 -> 28.8 mm
- net Net-(D13-A): track 0.00 -> 16.8 mm
- net Net-(Q3-D): track 0.00 -> 11.9 mm
- net Net-(Q2-B): track 0.00 -> 10.2 mm
Other:
- board size 246.8 x 135.9 mm -> 254.1 x 139.2 mm
